Commit message: robot motion success

File: robot_description/urdf/robot.urdf_.xacro (robot description, xacro)
@@ -1,10 +1,5 @@
 <?xml version="1.0"?>
 <robot xmlns:xacro="http://www.ros.org/wiki/xacro" name="3dof_robot">
-  <xacro:include filename="$(find robot_description)/urdf/robot_materials.xacro"/>
   <xacro:include filename="$(find robot_description)/urdf/robot_gazebo.xacro"/>
-  <xacro:red_material/>
-  <xacro:blue_material/>
-  <xacro:green_material/>
-  <xacro:gray_material/>
   <xacro:include filename="$(find robot_description)/urdf/robot_control.xacro"/>
   <xacro:include filename="$(find robot_description)/urdf/robot_materials.xacro"/>
@@ -43,5 +38,5 @@
           <cylinder radius="${radius}" length="${length}"/>
         </geometry>
-        <material name="gray_material"/>
+        <material><color rgba="${color}"/></material>
       </visual>
       <collision>
@@ -94,5 +89,5 @@
       <origin xyz="0.015 0 0.025" rpy="0 0 0"/>
       <geometry><box size="0.01 0.01 0.05"/></geometry>
-      <material name="gray_material"/>
+      <material><color rgba="0.2 0.2 0.2 1.0"/></material>
     </visual>
     <collision>
@@ -120,9 +115,8 @@
     </inertial>
   </link>
-  <joint name="link_4_to_gripper" type="revolute">
+  <joint name="link_4_to_gripper" type="fixed">
     <parent link="link_4"/>
     <child link="gripper_base"/>
     <origin xyz="0 0 ${l4}" rpy="0 0 0"/>
-    <limit lower="-1.57" upper="1.57" effort="50" velocity="1.0"/>
   </joint>
 </robot>

File: robot_description/urdf/robot_control.xacro (robot description, xacro)
@@ -7,4 +7,11 @@
         </hardware>
         <!-- Define Command and State interfaces for each joints -->
+        <joint name="link_4_to_gripper">
+            <command_interface name="position">
+                <param name="min">-${PI / 2}</param>
+                <param name="max">${PI / 2}</param>
+            </command_interface>
+            <state_interface name="position" />
+        </joint>
         <joint name="link_1_to_link_2">
             <command_interface name="position">

File: robot_description/urdf/robot_gazebo.xacro (robot description, xacro)
@@ -3,5 +3,5 @@
       <gazebo>
         <plugin filename="gz_ros2_control-system" name="gz_ros2_control::GazeboSimROS2ControlPlugin">
-            <parameters>$(find robot_description)/config/robot_controllers.yaml</parameters>
+            <parameters>$(find robot_controller)/config/robot_controllers.yaml</parameters>
         </plugin>
     </gazebo>
