Commit message: added nice visual for joints for rviz and gazebo

File: robot_description/urdf/robot.urdf.xacro (robot description, xacro)
@@ -3,18 +3,13 @@
   <xacro:include filename="$(find robot_description)/urdf/robot_materials.xacro"/>
   <xacro:include filename="$(find robot_description)/urdf/robot_gazebo.xacro"/>
-  <xacro:red_material/>
-  <xacro:blue_material/>
-  <xacro:green_material/>
-  <xacro:gray_material/>
   <xacro:include filename="$(find robot_description)/urdf/robot_control.xacro"/>
-  <xacro:include filename="$(find robot_description)/urdf/robot_materials.xacro"/>
   <!-- Link Parameters -->
-  <xacro:property name="r1" value="0.01"/>
-  <xacro:property name="r2" value="0.01"/>
-  <xacro:property name="r3" value="0.01"/>
-  <xacro:property name="r4" value="0.01"/>
-  <xacro:property name="l1" value="0.1"/>
-  <xacro:property name="l2" value="0.1"/>
-  <xacro:property name="l3" value="0.1"/>
+  <xacro:property name="r1" value="0.025"/>
+  <xacro:property name="r2" value="0.02"/>
+  <xacro:property name="r3" value="0.02"/>
+  <xacro:property name="r4" value="0.015"/>
+  <xacro:property name="l1" value="0.15"/>
+  <xacro:property name="l2" value="0.2"/>
+  <xacro:property name="l3" value="0.15"/>
   <xacro:property name="l4" value="0.1"/>
   <xacro:property name="m1" value="1.0"/>
@@ -22,4 +17,13 @@
   <xacro:property name="m3" value="0.6"/>
   <xacro:property name="m4" value="0.5"/>
+  <!-- Joint Visual Parameters -->
+  <xacro:property name="joint1_radius" value="0.05"/>
+  <xacro:property name="joint2_radius" value="0.020"/>
+  <xacro:property name="joint3_radius" value="0.020"/>
+  <xacro:property name="joint4_radius" value="0.020"/>
+  <xacro:property name="joint1_length" value="0.06"/>
+  <xacro:property name="joint2_length" value="0.05"/>
+  <xacro:property name="joint3_length" value="0.04"/>
+  <xacro:property name="joint4_length" value="0.04"/>
   <!-- Inertia macro for solid cylinder along Z-axis -->
   <xacro:macro name="inertial_cylinder_z" params="mass radius length">
@@ -43,5 +47,5 @@
           <cylinder radius="${radius}" length="${length}"/>
         </geometry>
-        <material name="gray_material"/>
+        <material name="${color}"/>
       </visual>
       <collision>
@@ -53,14 +57,50 @@
     </link>
   </xacro:macro>
-  <!-- World and Link 1 (Fixed) -->
+  <!-- Joint Visual Macro -->
+  <xacro:macro name="joint_visual" params="radius length">
+    <visual>
+      <origin xyz="0 0 0" rpy="0 0 0"/>
+      <geometry>
+        <cylinder radius="${radius}" length="${length}"/>
+      </geometry>
+      <material name="electric_blue"/>
+    </visual>
+  </xacro:macro>
+  <!-- Base -->
   <link name="world"/>
-  <xacro:cylinder_link name="link_1" mass="${m1}" radius="${r1}" length="${l1}" color="0.6 0.6 0.6 1.0"/>
-  <joint name="world_to_link_1" type="fixed">
+  <link name="base_link">
+    <visual>
+      <origin xyz="0 0 0.01" rpy="0 0 0"/>
+      <geometry>
+        <box size="0.2 0.2 0.02"/>
+      </geometry>
+      <material name="sleek_gray"/>
+    </visual>
+    <collision>
+      <origin xyz="0 0 0.01" rpy="0 0 0"/>
+      <geometry>
+        <box size="0.2 0.2 0.02"/>
+      </geometry>
+    </collision>
+    <inertial>
+      <origin xyz="0 0 0.01" rpy="0 0 0"/>
+      <mass value="2.0"/>
+      <inertia ixx="0.01" iyy="0.01" izz="0.01" ixy="0" ixz="0" iyz="0"/>
+    </inertial>
+  </link>
+  <joint name="world_to_base" type="fixed">
     <parent link="world"/>
+    <child link="base_link"/>
+    <origin xyz="0 0 0" rpy="0 0 0"/>
+  </joint>
+  <!-- Link 1 -->
+  <xacro:cylinder_link name="link_1" mass="${m1}" radius="${r1}" length="${l1}" color="metallic_silver"/>
+  <joint name="base_to_link_1" type="fixed">
+    <parent link="base_link"/>
     <child link="link_1"/>
-    <origin xyz="0 0 0" rpy="0 0 0"/>
-  </joint>
-  <!-- Link 2 -->
-  <xacro:cylinder_link name="link_2" mass="${m2}" radius="${r2}" length="${l2}" color="1.0 0.0 0.0 1.0"/>
+    <origin xyz="0 0 0.02" rpy="0 0 0"/>
+  </joint>
+  <!-- Link 2 with Joint Visual -->
+  <xacro:cylinder_link name="link_2" mass="${m2}" radius="${r2}" length="${l2}" color="deep_orange"/>
   <joint name="link_1_to_link_2" type="revolute">
     <parent link="link_1"/>
@@ -70,6 +110,14 @@
     <limit lower="-1.57" upper="1.57" effort="50" velocity="1.0"/>
   </joint>
-  <!-- Link 3 -->
-  <xacro:cylinder_link name="link_3" mass="${m3}" radius="${r3}" length="${l3}" color="0.0 0.7 1.0 1.0"/>
+  <link name="joint_1_visual">
+    <xacro:joint_visual radius="${joint1_radius}" length="${joint1_length}"/>
+  </link>
+  <joint name="joint_1_visual_joint" type="fixed">
+    <parent link="link_1"/>
+    <child link="joint_1_visual"/>
+    <origin xyz="0 0 ${l1}" rpy="${PI/2} 0 0"/>
+  </joint>
+  <!-- Link 3 with Joint Visual -->
+  <xacro:cylinder_link name="link_3" mass="${m3}" radius="${r3}" length="${l3}" color="metallic_silver"/>
   <joint name="link_2_to_link_3" type="revolute">
     <parent link="link_2"/>
@@ -79,6 +127,14 @@
     <limit lower="-1.57" upper="1.57" effort="50" velocity="1.0"/>
   </joint>
-  <!-- Link 4 -->
-  <xacro:cylinder_link name="link_4" mass="${m4}" radius="${r4}" length="${l4}" color="0.0 0.8 0.3 1.0"/>
+  <link name="joint_2_visual">
+    <xacro:joint_visual radius="${joint2_radius}" length="${joint2_length}"/>
+  </link>
+  <joint name="joint_2_visual_joint" type="fixed">
+    <parent link="link_2"/>
+    <child link="joint_2_visual"/>
+    <origin xyz="0 0 ${l2}" rpy="${PI/2} 0 0"/>
+  </joint>
+  <!-- Link 4 with Joint Visual -->
+  <xacro:cylinder_link name="link_4" mass="${m4}" radius="${r4}" length="${l4}" color="deep_orange"/>
   <joint name="link_3_to_link_4" type="revolute">
     <parent link="link_3"/>
@@ -88,35 +144,59 @@
     <limit lower="-1.57" upper="1.57" effort="50" velocity="1.0"/>
   </joint>
-  <!-- Gripper: Two Fingers Only -->
+  <link name="joint_3_visual">
+    <xacro:joint_visual radius="${joint3_radius}" length="${joint3_length}"/>
+  </link>
+  <joint name="joint_3_visual_joint" type="fixed">
+    <parent link="link_3"/>
+    <child link="joint_3_visual"/>
+    <origin xyz="0 0 ${l3}" rpy="${PI/2} 0 0"/>
+  </joint>
+  <!-- Gripper -->
   <link name="gripper_base">
-    <!-- Left Finger -->
-    <visual>
-      <origin xyz="0.015 0 0.025" rpy="0 0 0"/>
-      <geometry><box size="0.01 0.01 0.05"/></geometry>
-      <material name="gray_material"/>
-    </visual>
-    <collision>
-      <origin xyz="0.015 0 0.025" rpy="0 0 0"/>
-      <geometry><box size="0.01 0.01 0.05"/></geometry>
+    <visual>
+      <origin xyz="0 0 0.01" rpy="0 0 0"/>
+      <geometry>
+        <box size="0.04 0.03 0.02"/>
+      </geometry>
+      <material name="sleek_gray"/>
+    </visual>
+    <collision>
+      <origin xyz="0 0 0.01" rpy="0 0 0"/>
+      <geometry>
+        <box size="0.04 0.03 0.02"/>
+      </geometry>
     </collision>
     <inertial>
-      <origin xyz="0.015 0 0.025" rpy="0 0 0"/>
-      <mass value="0.025"/>
-      <inertia ixx="1e-5" iyy="1e-5" izz="1e-5" ixy="0" ixz="0" iyz="0"/>
+      <origin xyz="0 0 0.01" rpy="0 0 0"/>
+      <mass value="0.1"/>
+      <inertia ixx="1e-4" iyy="1e-4" izz="1e-4" ixy="0" ixz="0" iyz="0"/>
     </inertial>
-    <!-- Right Finger -->
-    <visual>
-      <origin xyz="-0.015 0 0.025" rpy="0 0 0"/>
-      <geometry><box size="0.01 0.01 0.05"/></geometry>
-    </visual>
-    <collision>
-      <origin xyz="-0.015 0 0.025" rpy="0 0 0"/>
-      <geometry><box size="0.01 0.01 0.05"/></geometry>
-    </collision>
-    <inertial>
-      <origin xyz="-0.015 0 0.025" rpy="0 0 0"/>
-      <mass value="0.025"/>
-      <inertia ixx="1e-5" iyy="1e-5" izz="1e-5" ixy="0" ixz="0" iyz="0"/>
-    </inertial>
+    <!-- Fingers -->
+    <visual>
+      <origin xyz="0.02 0 0.035" rpy="0 0 0"/>
+      <geometry>
+        <box size="0.01 0.015 0.05"/>
+      </geometry>
+      <material name="metallic_white"/>
+    </visual>
+    <collision>
+      <origin xyz="0.02 0 0.035" rpy="0 0 0"/>
+      <geometry>
+        <box size="0.01 0.015 0.05"/>
+      </geometry>
+    </collision>
+    <visual>
+      <origin xyz="-0.02 0 0.035" rpy="0 0 0"/>
+      <geometry>
+        <box size="0.01 0.015 0.05"/>
+      </geometry>
+      <material name="metallic_white"/>
+    </visual>
+    <collision>
+      <origin xyz="-0.02 0 0.035" rpy="0 0 0"/>
+      <geometry>
+        <box size="0.01 0.015 0.05"/>
+      </geometry>
+    </collision>
   </link>
   <joint name="link_4_to_gripper" type="revolute">
@@ -124,5 +204,14 @@
     <child link="gripper_base"/>
     <origin xyz="0 0 ${l4}" rpy="0 0 0"/>
-    <limit lower="-1.57" upper="1.57" effort="50" velocity="1.0"/>
+    <axis xyz="0 1 0"/>
+    <limit lower="-1.57" upper="1.57" effort="50" velocity="1.0"/>
+  </joint>
+  <link name="joint_4_visual">
+    <xacro:joint_visual radius="${joint4_radius}" length="${joint4_length}"/>
+  </link>
+  <joint name="joint_4_visual_joint" type="fixed">
+    <parent link="link_4"/>
+    <child link="joint_4_visual"/>
+    <origin xyz="0 0 ${l4}" rpy="${PI/2} 0 0"/>
   </joint>
 </robot>

File: robot_description/urdf/robot_materials.xacro (robot description, xacro)
@@ -1,27 +1,24 @@
 <?xml version="1.0"?>
-<robot xmlns:xacro="http://www.ros.org/wiki/xacro" name="3dof_robot">
-  <!-- Macro to define red material -->
-  <xacro:macro name="red_material" params="">
-    <material name="red_material">
-      <color rgba="0.8 0.1 0.1 1.0"/>
-    </material>
-  </xacro:macro>
-  <!-- Macro to define blue material -->
-  <xacro:macro name="blue_material" params="">
-    <material name="blue_material">
-      <color rgba="0.1 0.1 0.8 1.0"/>
-    </material>
-  </xacro:macro>
-  <!-- Macro to define green material -->
-  <xacro:macro name="green_material" params="">
-    <material name="green_material">
-      <color rgba="0.1 0.8 0.1 1.0"/>
-    </material>
-  </xacro:macro>
-  <!-- Macro to define gray material -->
-  <xacro:macro name="gray_material" params="">
-    <material name="gray_material">
-      <color rgba="0.5 0.5 0.5 1.0"/>
-    </material>
-  </xacro:macro>
+<robot xmlns:xacro="http://www.ros.org/wiki/xacro">
+  <!-- Material Definitions -->
+  <!-- Modern metallic silver for base and primary structure -->
+  <material name="metallic_silver">
+    <color rgba="0.8 0.8 0.85 1.0"/>
+  </material>
+  <!-- Deep orange accent for dynamic parts -->
+  <material name="deep_orange">
+    <color rgba="0.95 0.45 0.15 1.0"/>
+  </material>
+  <!-- Sleek dark gray for secondary parts -->
+  <material name="sleek_gray">
+    <color rgba="0.25 0.25 0.25 1.0"/>
+  </material>
+  <!-- Electric blue for joints and end-effector -->
+  <material name="electric_blue">
+    <color rgba="0.2 0.5 1.0 1.0"/>
+  </material>
+  <!-- Metallic white for highlights -->
+  <material name="metallic_white">
+    <color rgba="0.95 0.95 0.95 1.0"/>
+  </material>
 </robot>

Commit message: fixed joint dimentions and added joint tracking

File: robot_description/urdf/robot.urdf.xacro (robot description, xacro)
@@ -5,21 +5,21 @@
   <xacro:include filename="$(find robot_description)/urdf/robot_control.xacro"/>
   <!-- Link Parameters -->
-  <xacro:property name="r1" value="0.025"/>
-  <xacro:property name="r2" value="0.02"/>
-  <xacro:property name="r3" value="0.02"/>
-  <xacro:property name="r4" value="0.015"/>
-  <xacro:property name="l1" value="0.15"/>
-  <xacro:property name="l2" value="0.2"/>
-  <xacro:property name="l3" value="0.15"/>
-  <xacro:property name="l4" value="0.1"/>
-  <xacro:property name="m1" value="1.0"/>
-  <xacro:property name="m2" value="0.8"/>
-  <xacro:property name="m3" value="0.6"/>
-  <xacro:property name="m4" value="0.5"/>
+  <xacro:property name="r1" value="0.024"/>   <!-- Base link radius -->
+  <xacro:property name="r2" value="0.020"/>  <!-- Second link radius -->
+  <xacro:property name="r3" value="0.020"/>   <!-- Third link radius -->
+  <xacro:property name="r4" value="0.015"/>  <!-- End effector radius -->
+  <xacro:property name="l1" value="0.25"/>    <!-- Base link length -->
+  <xacro:property name="l2" value="0.15"/>   <!-- Second link length -->
+  <xacro:property name="l3" value="0.15"/>    <!-- Third link length -->
+  <xacro:property name="l4" value="0.10"/>   <!-- End effector length -->
+  <xacro:property name="m1" value="0.8"/>    <!-- Base link mass -->
+  <xacro:property name="m2" value="0.6"/>    <!-- Second link mass -->
+  <xacro:property name="m3" value="0.4"/>    <!-- Third link mass -->
+  <xacro:property name="m4" value="0.3"/>    <!-- End effector mass -->
   <!-- Joint Visual Parameters -->
-  <xacro:property name="joint1_radius" value="0.05"/>
+  <xacro:property name="joint1_radius" value="0.035"/>
   <xacro:property name="joint2_radius" value="0.020"/>
   <xacro:property name="joint3_radius" value="0.020"/>
-  <xacro:property name="joint4_radius" value="0.020"/>
+  <xacro:property name="joint4_radius" value="0.013"/>
   <xacro:property name="joint1_length" value="0.06"/>
   <xacro:property name="joint2_length" value="0.05"/>

File: robot_description/urdf/robot_control.xacro (robot description, xacro)
@@ -8,30 +8,26 @@
         <!-- Define Command and State interfaces for each joints -->
         <joint name="link_4_to_gripper">
-            <command_interface name="position">
-                <param name="min">-${PI / 2}</param>
-                <param name="max">${PI / 2}</param>
-            </command_interface>
-            <state_interface name="position" />
+            <command_interface name="effort"/>
+            <state_interface name="position"/>
+            <state_interface name="velocity"/>
+            <state_interface name="effort"/>
         </joint>
         <joint name="link_1_to_link_2">
-            <command_interface name="position">
-                <param name="min">-${PI / 2}</param>
-                <param name="max">${PI / 2}</param>
-            </command_interface>
-            <state_interface name="position" />
+            <command_interface name="effort"/>
+            <state_interface name="position"/>
+            <state_interface name="velocity"/>
+            <state_interface name="effort"/>
         </joint>
         <joint name="link_2_to_link_3">
-            <command_interface name="position">
-                <param name="min">-${PI / 2}</param>
-                <param name="max">${PI / 2}</param>
-            </command_interface>
-            <state_interface name="position" />
+            <command_interface name="effort"/>
+            <state_interface name="position"/>
+            <state_interface name="velocity"/>
+            <state_interface name="effort"/>
         </joint>
         <joint name="link_3_to_link_4">
-            <command_interface name="position">
-                <param name="min">-${PI / 2}</param>
-                <param name="max">${PI / 2}</param>
-            </command_interface>
-            <state_interface name="position" />
+            <command_interface name="effort"/>
+            <state_interface name="position"/>
+            <state_interface name="velocity"/>
+            <state_interface name="effort"/>
         </joint>
     </ros2_control>

Commit message: positio command and postion and velocity as state interface

File: robot_description/urdf/robot.urdf.xacro (robot description, xacro)
@@ -1,4 +1,6 @@
 <?xml version="1.0"?>
 <robot xmlns:xacro="http://www.ros.org/wiki/xacro" name="3dof_robot">
+  <!-- Define PI constant -->
+  <xacro:property name="PI" value="3.14159265359"/>
   <xacro:include filename="$(find robot_description)/urdf/robot_materials.xacro"/>
   <xacro:include filename="$(find robot_description)/urdf/robot_gazebo.xacro"/>

File: robot_description/urdf/robot_control.xacro (robot description, xacro)
@@ -1,34 +1,75 @@
 <?xml version="1.0"?>
 <robot xmlns:xacro="http://www.ros.org/wiki/xacro" name="3dof_robot">
+    <!-- Define PI constant -->
+    <xacro:property name="PI" value="3.14159265359"/>
     <ros2_control name="RobotSystem" type="system">
-        <xacro:property name="PI" value="3.14159265359" />
         <hardware>
             <plugin>gz_ros2_control/GazeboSimSystem</plugin>
         </hardware>
-        <!-- Define Command and State interfaces for each joints -->
-        <joint name="link_4_to_gripper">
-            <command_interface name="effort"/>
+        <!-- Base Joint -->
+        <joint name="link_1_to_link_2">
+            <command_interface name="position"/>
             <state_interface name="position"/>
             <state_interface name="velocity"/>
-            <state_interface name="effort"/>
+            <param name="initial_position">0.0</param>
         </joint>
-        <joint name="link_1_to_link_2">
-            <command_interface name="effort"/>
+        <!-- Shoulder Joint -->
+        <joint name="link_2_to_link_3">
+            <command_interface name="position"/>
             <state_interface name="position"/>
             <state_interface name="velocity"/>
-            <state_interface name="effort"/>
+            <param name="initial_position">0.0</param>
         </joint>
-        <joint name="link_2_to_link_3">
-            <command_interface name="effort"/>
+        <!-- Elbow Joint -->
+        <joint name="link_3_to_link_4">
+            <command_interface name="position"/>
             <state_interface name="position"/>
             <state_interface name="velocity"/>
-            <state_interface name="effort"/>
+            <param name="initial_position">0.0</param>
         </joint>
-        <joint name="link_3_to_link_4">
-            <command_interface name="effort"/>
+        <!-- Gripper Joint -->
+        <joint name="link_4_to_gripper">
+            <command_interface name="position"/>
             <state_interface name="position"/>
             <state_interface name="velocity"/>
-            <state_interface name="effort"/>
+            <param name="initial_position">0.0</param>
         </joint>
     </ros2_control>
+    <!-- Transmissions -->
+    <transmission name="link_1_to_link_2_trans">
+        <type>transmission_interface/SimpleTransmission</type>
+        <joint name="link_1_to_link_2">
+            <hardwareInterface>hardware_interface/PositionJointInterface</hardwareInterface>
+        </joint>
+        <actuator name="link_1_to_link_2_motor">
+            <mechanicalReduction>1</mechanicalReduction>
+        </actuator>
+    </transmission>
+    <transmission name="link_2_to_link_3_trans">
+        <type>transmission_interface/SimpleTransmission</type>
+        <joint name="link_2_to_link_3">
+            <hardwareInterface>hardware_interface/PositionJointInterface</hardwareInterface>
+        </joint>
+        <actuator name="link_2_to_link_3_motor">
+            <mechanicalReduction>1</mechanicalReduction>
+        </actuator>
+    </transmission>
+    <transmission name="link_3_to_link_4_trans">
+        <type>transmission_interface/SimpleTransmission</type>
+        <joint name="link_3_to_link_4">
+            <hardwareInterface>hardware_interface/PositionJointInterface</hardwareInterface>
+        </joint>
+        <actuator name="link_3_to_link_4_motor">
+            <mechanicalReduction>1</mechanicalReduction>
+        </actuator>
+    </transmission>
+    <transmission name="link_4_to_gripper_trans">
+        <type>transmission_interface/SimpleTransmission</type>
+        <joint name="link_4_to_gripper">
+            <hardwareInterface>hardware_interface/PositionJointInterface</hardwareInterface>
+        </joint>
+        <actuator name="link_4_to_gripper_motor">
+            <mechanicalReduction>1</mechanicalReduction>
+        </actuator>
+    </transmission>
 </robot>
